File: src/CYPD3177_Power-Board.kicad_sch (KiCad schematic)
At the start: 48 parts, among them J1 Conn_01x06, J2 USB4125-GF-A, J3 Conn_01x03, J4 Conn_01x03, J5 Conn_01x03, Q1 IRF9358PbF, Q2 BSL308PE, Q3 NTR4503N, U1 CYPD3177-24LQXQx

Commit message: Mod: Schematic and database, changed LCSC part number of R3
Parts:
- R3: LCSC C60490 -> C106231
Changed lines of the file:
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@@
       (effects (font (size 1.27 1.27)) hide)
     )
-    (property "LCSC" "C60490" (at 199.39 42.545 0)
+    (property "LCSC" "C106231" (at 199.39 42.545 0)
       (effects (font (size 1.27 1.27)) hide)
     )
